File: Eagle/Serqet/Serqet.brd (EAGLE design)
At the start: 160 x 100 mm, 65 parts

Commit message: Added board dim.  Added board cruft to git ignore
Other:
- board size 160 x 100 mm -> 127 x 43.2 mm
Changed lines of the file:
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@@
 <board>
 <plain>
-<wire x1="0" y1="0" x2="160" y2="0" width="0" layer="20"/>
-<wire x1="160" y1="0" x2="160" y2="100" width="0" layer="20"/>
-<wire x1="160" y1="100" x2="0" y2="100" width="0" layer="20"/>
-<wire x1="0" y1="100" x2="0" y2="0" width="0" layer="20"/>
+<wire x1="0" y1="0" x2="127" y2="0" width="0.4064" layer="20"/>
+<wire x1="127" y1="0" x2="127" y2="43.18" width="0.4064" layer="20"/>
+<wire x1="127" y1="43.18" x2="0" y2="43.18" width="0.4064" layer="20"/>
+<wire x1="0" y1="43.18" x2="0" y2="0" width="0.4064" layer="20"/>
 </plain>
 <attributes>
